File: PD Smart Supply.kicad_pcb (KiCad board)
At the start: 2 copper layers, 67 parts, among them P1 WJ500V-5.08-2P-14-00A, P2 WJ500V-5.08-2P-14-00A, Q1 2N7002, Q2 2N7002, SW1 Switch, SW2 Rotary Encoder, U1 CH224A, U2 TPS560430XDBVR, U3 STM32G071CBT6, U4 TPS259470LRPWR, U5 OLED

Commit message: Complete Rev A PCB layout and manufacturing preparation
Finalize the four-layer placement, routing, ground pours, silkscreen branding, connector labels, and test-point markings.

Add board design rules, fabrication toolkit settings, project documentation, and ignore regenerable plugin outputs.
Parts:
- removed R23, R24, R25: 1KΩ, PD Smart Supply:R0402
- added R26: 10KΩ, PD Smart Supply:R0402, F.Cu at (113.3, 95.5)
- added R27: 10KΩ, PD Smart Supply:R0402, F.Cu at (120.7, 95.3)
- added R28: 10KΩ, PD Smart Supply:R0402, F.Cu at (128.0, 95.3)
- added REF**: MountingHole_3.2mm_M3, MountingHole:MountingHole_3.2mm_M3, F.Cu at (165.5, 95.5)
- added REF**: MountingHole_3.2mm_M3, MountingHole:MountingHole_3.2mm_M3, F.Cu at (104.5, 95.5)
- added REF**: MountingHole_3.2mm_M3, MountingHole:MountingHole_3.2mm_M3, F.Cu at (165.5, 54.5)
- added REF**: MountingHole_3.2mm_M3, MountingHole:MountingHole_3.2mm_M3, F.Cu at (104.5, 54.5)
- added SW3: UP, PD Smart Supply:SW-SMD_XYECONN_TSC01-TBW0FH3.5, F.Cu at (111.6, 98.0)
- added SW4: Select, PD Smart Supply:SW-SMD_XYECONN_TSC01-TBW0FH3.5, F.Cu at (126.3, 98.0)
- SW2: value Rotary Encoder -> Down; footprint PD Smart Supply:SW-SMD_EC11J1525402 -> PD Smart Supply:SW-SMD_XYECONN_TSC01-TBW0FH3.5
- TP_3V3: value TestPoint -> 3V3; footprint PD Smart Supply:D0402-BI -> TestPoint:TestPoint_Pad_D1.0mm
- TP_GND1: value TestPoint -> GND; footprint TestPoint:TestPoint_Pad_D1.5mm -> TestPoint:TestPoint_Pad_D1.0mm
- TP_ISENSE1: value TestPoint -> ISENSE; footprint TestPoint:TestPoint_Pad_D1.5mm -> TestPoint:TestPoint_Pad_D1.0mm
- TP_VBUS_PD1: value TestPoint -> VBUS; footprint TestPoint:TestPoint_Pad_D1.5mm -> TestPoint:TestPoint_Pad_D1.0mm
- TP_VOUT1: value TestPoint -> VOUT; footprint TestPoint:TestPoint_Pad_D1.5mm -> TestPoint:TestPoint_Pad_D1.0mm
- TP_VSENSE1: value TestPoint -> VSENSE; footprint TestPoint:TestPoint_Pad_D1.5mm -> TestPoint:TestPoint_Pad_D1.0mm
- moved U5 232.8 mm to (101.8, 75.0), turned to 90 degrees
- moved L1 231.8 mm to (136.5, 81.3), turned to 90 degrees
- moved TP_3V3 231.5 mm to (136.1, 76.8)
- moved C14 229.0 mm to (135.7, 58.3), turned to 180 degrees
- moved R10 227.3 mm to (138.1, 73.2), turned to -90 degrees
- moved R5 225.8 mm to (138.7, 94.6), turned to -90 degrees
- moved LED1 224.5 mm to (143.7, 97.7)
- moved R9 224.0 mm to (138.1, 75.4), turned to 90 degrees
- moved C7 223.5 mm to (130.4, 84.0), turned to -90 degrees
- moved C16 223.4 mm to (142.3, 54.2), turned to 90 degrees
- moved U2 223.2 mm to (134.1, 88.1), turned to -90 degrees
- moved R19 221.4 mm to (144.0, 59.6)
- moved C13 221.2 mm to (135.7, 70.9), turned to 90 degrees
- moved R16 221.2 mm to (144.0, 61.3), turned to 180 degrees
- moved C2 219.5 mm to (143.6, 84.4), turned to 90 degrees
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Connections:
- net Net-(U2-SW) renamed /BUCK_SW
- U3 pad 17: /ENC_A -> /BTN_UP
- U3 pad 18: /ENC_B -> /BTN_DOWN
- U3 pad 19: /ENC_SW -> /BTN_SELECT
- USB1 pad A5: Net-(U1-CC2) -> Net-(U1-CC1)
- USB1 pad B5: Net-(U1-CC1) -> Net-(U1-CC2)
Routing:
- net +3.3V: track 0.00 -> 160.2 mm, vias 0 -> 7
- net /VBUS_PD: track 0.00 -> 95.1 mm, vias 0 -> 4
- net GND: track 0.00 -> 88.7 mm, vias 0 -> 35
- net /NRST: track 0.00 -> 87.9 mm, vias 0 -> 6
- net /BTN_UP: track 0.00 -> 78.2 mm, vias 0 -> 4
- net /BTN_SELECT: track 0.00 -> 76.9 mm, vias 0 -> 4
- net /BTN_DOWN: track 0.00 -> 68.7 mm, vias 0 -> 4
- net /PG: track 0.00 -> 50.5 mm, vias 0 -> 4
- net /EFUSE_OUT: track 0.00 -> 45.1 mm
- net /SWCLK: track 0.00 -> 42.7 mm, vias 0 -> 2
- net /OLED_SDA: track 0.00 -> 41.6 mm, vias 0 -> 2
- net /OLED_SCL: track 0.00 -> 39.6 mm
- net /CFG2: track 0.00 -> 35.1 mm, vias 0 -> 2
- net /CFG1: track 0.00 -> 35.0 mm, vias 0 -> 3
- net /CFG3: track 0.00 -> 34.1 mm, vias 0 -> 2
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- added copper zone on F.Cu, net +3.3V
- added copper zone on F.Cu, net /BUCK_SW
- added copper zone on F.Cu, net /EFUSE_OUT
- added copper zone on F.Cu, net /VBUS_PD
- added copper zone on F.Cu, net GND
- added copper zone on In1.Cu, net GND
- added copper zone on In2.Cu, net GND
Other:
- board outline added: 70 x 50 mm
- copper layers 2 -> 4
- board text added: "+"
- board text added: "-"
- board text added: "DW"
- board text added: "Designed by Yafet Daniel"
- board text added: "GND"
- board text added: "NRST"
- board text added: "OK"
- board text added: "OUT1"
- board text added: "OUT2"
- board text added: "PD SMART SUPPLY"
- board text added: "REV A • 2026-08"
- board text added: "RST"
- board text added: "SWCLK"
- board text added: "SWDIO"
- board text added: "UP"

Commit message: Finalize Rev A design for manufacturing
Synchronize final component metadata and fabrication settings, preserve the completed PCB state, add the Rev A design record, and organize simulation and calculator references under Docs.
Parts:
- SW1: value Switch -> TSC01-TBW0FH3.5
- SW2: value Down -> TSC01-TBW0FH3.5
- SW3: value UP -> TSC01-TBW0FH3.5
- SW4: value Select -> TSC01-TBW0FH3.5
- U5: value OLED -> HS96L03W2C03
Changed lines of the file:
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@@
 			)
 		)
-		(property "Value" "Switch"
+		(property "Value" "TSC01-TBW0FH3.5"
 			(at 0 4.725 0)
 			(layer "F.Fab")
@@
 			)
 		)
-		(property "Value" "UP"
+		(property "Value" "TSC01-TBW0FH3.5"
 			(at 0 4.725 0)
 			(layer "F.Fab")
@@
 			)
 		)
-		(property "Value" "Select"
+		(property "Value" "TSC01-TBW0FH3.5"
 			(at 0 4.725 0)
 			(layer "F.Fab")
@@
 			)
 		)
-		(property "Value" "Down"
+		(property "Value" "TSC01-TBW0FH3.5"
 			(at 0 4.725 0)
 			(layer "F.Fab")
@@
 			)
 		)
-		(property "Value" "OLED"
+		(property "Value" "HS96L03W2C03"
 			(at 0 4 90)
 			(layer "F.Fab")
